File: hardware/artemis-synth-v1.sch (KiCad schematic (older format))
At the start: 55 parts, among them IC1 ATMEGA328P, J1 USB_2_MB, J2 AVR-ISP-6, SW10 SWITCH_PUSH_CW, SW11 SWITCH_PUSH_CW, SW2 SWITCH_PUSH_CW, SW3 SWITCH_PUSH_CW, SW4 SWITCH_PUSH_CW, SW5 SWITCH_PUSH_CW, SW6 SWITCH_PUSH_CW, SW7 SWITCH_PUSH_CW, SW8 SWITCH_PUSH_CW, SW9 SWITCH_PUSH_CW, U1 MCP4921, U2 TDA2722M, X1 16MHz

Commit message: Fixed drill file and change USB connector footprint
Parts:
- removed J1: USB_2_MB, SparkFun-USB-MB-H, symbol USB_2_MB
- added J1: USB_2, USB_B, symbol USB_2
Connections:
- no-connect marks 2 -> 1

Commit message: Made BOM, fixed up board. submitting to Eric for review
Parts:
- R4: value 50K -> 47K
Changed lines of the file:
@@
-EESchema Schematic File Version 2  date Mon 02 Jul 2012 09:39:48 AM EDT
+EESchema Schematic File Version 2  date Mon 02 Jul 2012 02:20:01 PM EDT
 LIBS:power
 LIBS:device
@@
 Optoloader\n
 $Comp
-L +3.3V #PWR21
+L +3.3V #PWR01
 U 1 1 4FE933FC
 P 6775 3325
-F 0 "#PWR21" H 6775 3285 30  0001 C CNN
+F 0 "#PWR01" H 6775 3285 30  0001 C CNN
 F 1 "+3.3V" H 6775 3435 30  0000 C CNN
 	1    6775 3325
@@
 $EndComp
 $Comp
-L +3.3V #PWR23
+L +3.3V #PWR02
 U 1 1 4FE933CC
 P 7100 3325
-F 0 "#PWR23" H 7100 3285 30  0001 C CNN
+F 0 "#PWR02" H 7100 3285 30  0001 C CNN
 F 1 "+3.3V" H 7100 3435 30  0000 C CNN
 	1    7100 3325
@@
 $EndComp
 $Comp
-L GND #PWR24
+L GND #PWR03
 U 1 1 4FE933C5
 P 7100 4850
-F 0 "#PWR24" H 7100 4850 30  0001 C CNN
+F 0 "#PWR03" H 7100 4850 30  0001 C CNN
 F 1 "GND" H 7100 4780 30  0001 C CNN
 	1    7100 4850
@@
 XTAL2
 $Comp
-L GND #PWR2
+L GND #PWR04
 U 1 1 4FE92692
 P 825 3800
-F 0 "#PWR2" H 825 3800 30  0001 C CNN
+F 0 "#PWR04" H 825 3800 30  0001 C CNN
 F 1 "GND" H 825 3730 30  0001 C CNN
 	1    825  3800
@@
 L0
 $Comp
-L +3.3V #PWR40
+L +3.3V #PWR05
 U 1 1 4FE92549
 P 10400 4125
-F 0 "#PWR40" H 10400 4085 30  0001 C CNN
+F 0 "#PWR05" H 10400 4085 30  0001 C CNN
 F 1 "+3.3V" H 10400 4235 30  0000 C CNN
 	1    10400 4125
@@
 $EndComp
 $Comp
-L +3.3V #PWR37
+L +3.3V #PWR06
 U 1 1 4FE92545
 P 10025 4125
-F 0 "#PWR37" H 10025 4085 30  0001 C CNN
+F 0 "#PWR06" H 10025 4085 30  0001 C CNN
 F 1 "+3.3V" H 10025 4235 30  0000 C CNN
 	1    10025 4125
@@
 $EndComp
 $Comp
-L +3.3V #PWR34
+L +3.3V #PWR07
 U 1 1 4FE92541
 P 9700 4125
-F 0 "#PWR34" H 9700 4085 30  0001 C CNN
+F 0 "#PWR07" H 9700 4085 30  0001 C CNN
 F 1 "+3.3V" H 9700 4235 30  0000 C CNN
 	1    9700 4125
@@
 $EndComp
 $Comp
-L +3.3V #PWR30
+L +3.3V #PWR08
 U 1 1 4FE92538
 P 9375 4125
-F 0 "#PWR30" H 9375 4085 30  0001 C CNN
+F 0 "#PWR08" H 9375 4085 30  0001 C CNN
 F 1 "+3.3V" H 9375 4235 30  0000 C CNN
 	1    9375 4125
@@
 $EndComp
 $Comp
-L GND #PWR41
+L GND #PWR09
 U 1 1 4FE92533
 P 10400 5275
-F 0 "#PWR41" H 10400 5275 30  0001 C CNN
+F 0 "#PWR09" H 10400 5275 30  0001 C CNN
 F 1 "GND" H 10400 5205 30  0001 C CNN
 	1    10400 5275
@@
 $EndComp
 $Comp
-L GND #PWR38
+L GND #PWR010
 U 1 1 4FE9252F
 P 10025 5275
-F 0 "#PWR38" H 10025 5275 30  0001 C CNN
+F 0 "#PWR010" H 10025 5275 30  0001 C CNN
 F 1 "GND" H 10025 5205 30  0001 C CNN
 	1    10025 5275
@@
 $EndComp
 $Comp
-L GND #PWR35
+L GND #PWR011
 U 1 1 4FE92526
 P 9700 5275
-F 0 "#PWR35" H 9700 5275 30  0001 C CNN
+F 0 "#PWR011" H 9700 5275 30  0001 C CNN
 F 1 "GND" H 9700 5205 30  0001 C CNN
 	1    9700 5275
@@
 $EndComp
 $Comp
-L GND #PWR31
+L GND #PWR012
 U 1 1 4FE92521
 P 9375 5275
-F 0 "#PWR31" H 9375 5275 30  0001 C CNN
+F 0 "#PWR012" H 9375 5275 30  0001 C CNN
 F 1 "GND" H 9375 5205 30  0001 C CNN
 	1    9375 5275
@@
 $EndComp
 $Comp
-L GND #PWR14
+L GND #PWR013
 U 1 1 4FE8F262
 P 5250 7575
-F 0 "#PWR14" H 5250 7575 30  0001 C CNN
+F 0 "#PWR013" H 5250 7575 30  0001 C CNN
 F 1 "GND" H 5250 7505 30  0001 C CNN
 	1    5250 7575
@@
 BT0
 $Comp
-L GND #PWR11
+L GND #PWR014
 U 1 1 4FE8F01C
 P 4125 7550
-F 0 "#PWR11" H 4125 7550 30  0001 C CNN
+F 0 "#PWR014" H 4125 7550 30  0001 C CNN
 F 1 "GND" H 4125 7480 30  0001 C CNN
 	1    4125 7550
@@
 $EndComp
 $Comp
-L +3.3V #PWR18
+L +3.3V #PWR015
 U 1 1 4FE8EEC3
 P 6675 1050
-F 0 "#PWR18" H 6675 1010 30  0001 C CNN
+F 0 "#PWR015" H 6675 1010 30  0001 C CNN
 F 1 "+3.3V" H 6675 1160 30  0000 C CNN
 	1    6675 1050
@@
 $EndComp
 $Comp
-L +3.3V #PWR10
+L +3.3V #PWR016
 U 1 1 4FE8EEBE
 P 3175 1575
-F 0 "#PWR10" H 3175 1535 30  0001 C CNN
+F 0 "#PWR016" H 3175 1535 30  0001 C CNN
 F 1 "+3.3V" H 3175 1685 30  0000 C CNN
 	1    3175 1575
@@
 $EndComp
 $Comp
-L +3.3V #PWR3
+L +3.3V #PWR017
 U 1 1 4FE8EEBA
 P 1300 1100
-F 0 "#PWR3" H 1300 1060 30  0001 C CNN
+F 0 "#PWR017" H 1300 1060 30  0001 C CNN
 F 1 "+3.3V" H 1300 1210 30  0000 C CNN
 	1    1300 1100
@@
 $EndComp
 $Comp
-L +3.3V #PWR12
+L +3.3V #PWR018
 U 1 1 4FE8EEAB
 P 4700 775
-F 0 "#PWR12" H 4700 735 30  0001 C CNN
+F 0 "#PWR018" H 4700 735 30  0001 C CNN
 F 1 "+3.3V" H 4700 885 30  0000 C CNN
 	1    4700 775
@@
 $EndComp
 $Comp
-L GND #PWR4
+L GND #PWR019
 U 1 1 4FE8EE66
 P 1300 2000
-F 0 "#PWR4" H 1300 2000 30  0001 C CNN
+F 0 "#PWR019" H 1300 2000 30  0001 C CNN
 F 1 "GND" H 1300 1930 30  0001 C CNN
 	1    1300 2000
@@
 USBasp Bootloader Interface\n
 $Comp
-L GND #PWR7
+L GND #PWR020
 U 1 1 4FE60A89
 P 2025 5250
-F 0 "#PWR7" H 2025 5250 30  0001 C CNN
+F 0 "#PWR020" H 2025 5250 30  0001 C CNN
 F 1 "GND" H 2025 5180 30  0001 C CNN
 	1    2025 5250
@@
 $EndComp
 $Comp
-L GND #PWR6
+L GND #PWR021
 U 1 1 4FE60A82
 P 1725 5250
-F 0 "#PWR6" H 1725 5250 30  0001 C CNN
+F 0 "#PWR021" H 1725 5250 30  0001 C CNN
 F 1 "GND" H 1725 5180 30  0001 C CNN
 	1    1725 5250
@@
 $EndComp
 $Comp
-L GND #PWR5
+L GND #PWR022
 U 1 1 4FE609B3
 P 1475 4900
-F 0 "#PWR5" H 1475 4900 30  0001 C CNN
+F 0 "#PWR022" H 1475 4900 30  0001 C CNN
 F 1 "GND" H 1475 4830 30  0001 C CNN
 	1    1475 4900
@@
 $EndComp
 $Comp
-L GND #PWR8
+L GND #PWR023
 U 1 1 4FE5FE71
 P 2675 2150
-F 0 "#PWR8" H 2675 2150 30  0001 C CNN
+F 0 "#PWR023" H 2675 2150 30  0001 C CNN
 F 1 "GND" H 2675 2080 30  0001 C CNN
 	1    2675 2150
@@
 $EndComp
 $Comp
-L GND #PWR39
+L GND #PWR024
 U 1 1 4FE4E2CA
 P 10175 3150
-F 0 "#PWR39" H 10175 3150 30  0001 C CNN
+F 0 "#PWR024" H 10175 3150 30  0001 C CNN
 F 1 "GND" H 10175 3080 30  0001 C CNN
 	1    10175 3150
@@
 $EndComp
 $Comp
-L GND #PWR42
+L GND #PWR025
 U 1 1 4FE4E2C1
 P 10475 3150
-F 0 "#PWR42" H 10475 3150 30  0001 C CNN
+F 0 "#PWR025" H 10475 3150 30  0001 C CNN
 F 1 "GND" H 10475 3080 30  0001 C CNN
 	1    10475 3150
@@
 $EndComp
 $Comp
-L GND #PWR27
+L GND #PWR026
 U 1 1 4FE4E282
 P 8125 2000
-F 0 "#PWR27" H 8125 2000 30  0001 C CNN
+F 0 "#PWR026" H 8125 2000 30  0001 C CNN
 F 1 "GND" H 8125 1930 30  0001 C CNN
 	1    8125 2000
@@
 $EndComp
 $Comp
-L GND #PWR26
+L GND #PWR027
 U 1 1 4FE4E267
 P 7875 2725
-F 0 "#PWR26" H 7875 2725 30  0001 C CNN
+F 0 "#PWR027" H 7875 2725 30  0001 C CNN
 F 1 "GND" H 7875 2655 30  0001 C CNN
 	1    7875 2725
@@
 $EndComp
 $Comp
-L GND #PWR29
+L GND #PWR028
 U 1 1 4FE4E1B5
 P 8675 2175
-F 0 "#PWR29" H 8675 2175 30  0001 C CNN
+F 0 "#PWR028" H 8675 2175 30  0001 C CNN
 F 1 "GND" H 8675 2105 30  0001 C CNN
 	1    8675 2175
@@
 $EndComp
 $Comp
-L GND #PWR28
+L GND #PWR029
 U 1 1 4FE4E1A2
 P 8375 2725
-F 0 "#PWR28" H 8375 2725 30  0001 C CNN
+F 0 "#PWR029" H 8375 2725 30  0001 C CNN
 F 1 "GND" H 8375 2655 30  0001 C CNN
 	1    8375 2725
@@
 $EndComp
 $Comp
-L GND #PWR16
+L GND #PWR030
 U 1 1 4FE4C40C
 P 5825 2425
-F 0 "#PWR16" H 5825 2425 30  0001 C CNN
+F 0 "#PWR030" H 5825 2425 30  0001 C CNN
 F 1 "GND" H 5825 2355 30  0001 C CNN
 	1    5825 2425
@@
 $EndComp
 $Comp
-L GND #PWR17
+L GND #PWR031
 U 1 1 4FDE504C
 P 6175 1750
-F 0 "#PWR17" H 6175 1750 30  0001 C CNN
+F 0 "#PWR031" H 6175 1750 30  0001 C CNN
 F 1 "GND" H 6175 1680 30  0001 C CNN
 	1    6175 1750
@@
 $EndComp
 $Comp
-L GND #PWR36
+L GND #PWR032
 U 1 1 4FDE49E8
 P 9975 1150
-F 0 "#PWR36" H 9975 1150 30  0001 C CNN
+F 0 "#PWR032" H 9975 1150 30  0001 C CNN
 F 1 "GND" H 9975 1080 30  0001 C CNN
 	1    9975 1150
@@
 $EndComp
 $Comp
-L GND #PWR25
+L GND #PWR033
 U 1 1 4FDE499C
 P 7325 1750
-F 0 "#PWR25" H 7325 1750 30  0001 C CNN
+F 0 "#PWR033" H 7325 1750 30  0001 C CNN
 F 1 "GND" H 7325 1680 30  0001 C CNN
 	1    7325 1750
@@
 CS/
 $Comp
-L GND #PWR20
+L GND #PWR034
 U 1 1 4FDC0B04
 P 6775 2825
-F 0 "#PWR20" H 6775 2825 30  0001 C CNN
+F 0 "#PWR034" H 6775 2825 30  0001 C CNN
 F 1 "GND" H 6775 2755 30  0001 C CNN
 	1    6775 2825
@@
 $EndComp
 $Comp
-L GND #PWR33
+L GND #PWR035
 U 1 1 4FDC080E
 P 9475 2975
-F 0 "#PWR33" H 9475 2975 30  0001 C CNN
+F 0 "#PWR035" H 9475 2975 30  0001 C CNN
 F 1 "GND" H 9475 2905 30  0001 C CNN
 	1    9475 2975
@@
 $EndComp
 $Comp
-L GND #PWR9
+L GND #PWR036
 U 1 1 4FDC0519
 P 3125 4225
-F 0 "#PWR9" H 3125 4225 30  0001 C CNN
+F 0 "#PWR036" H 3125 4225 30  0001 C CNN
 F 1 "GND" H 3125 4155 30  0001 C CNN
 	1    3125 4225
@@
 MOSI
 $Comp
-L GND #PWR13
+L GND #PWR037
 U 1 1 4FDAC48B
 P 4700 1475
-F 0 "#PWR13" H 4700 1475 30  0001 C CNN
+F 0 "#PWR037" H 4700 1475 30  0001 C CNN
 F 1 "GND" H 4700 1405 30  0001 C CNN
 	1    4700 1475
@@
 $EndComp
 $Comp
-L GND #PWR1
+L GND #PWR038
 U 1 1 4FEA30E8
 P 700 4350
-F 0 "#PWR1" H 700 4350 30  0001 C CNN
+F 0 "#PWR038" H 700 4350 30  0001 C CNN
 F 1 "GND" H 700 4280 30  0001 C CNN
 	1    700  4350
@@
 $EndComp
 $Comp
-L +3.3V #PWR15
+L +3.3V #PWR039
 U 1 1 4FEA50E6
 P 5525 2725
-F 0 "#PWR15" H 5525 2685 30  0001 C CNN
+F 0 "#PWR039" H 5525 2685 30  0001 C CNN
 F 1 "+3.3V" H 5525 2835 30  0000 C CNN
 	1    5525 2725
@@
 $EndComp
 $Comp
-L GND #PWR22
+L GND #PWR040
 U 1 1 4FEA58E6
 P 6775 4850
-F 0 "#PWR22" H 6775 4850 30  0001 C CNN
+F 0 "#PWR040" H 6775 4850 30  0001 C CNN
 F 1 "GND" H 6775 4780 30  0001 C CNN
 	1    6775 4850
@@
 $EndComp
 $Comp
-L +3.3V #PWR19
+L +3.3V #PWR041
 U 1 1 4FEA5D07
 P 6775 1600
-F 0 "#PWR19" H 6775 1560 30  0001 C CNN
+F 0 "#PWR041" H 6775 1560 30  0001 C CNN
 F 1 "+3.3V" H 6775 1710 30  0000 C CNN
 	1    6775 1600
@@
 2xAA Batteries (Switch on battery holder)
 $Comp
-L +3.3V #PWR32
+L +3.3V #PWR042
 U 1 1 4FEA8074
 P 9475 1050
-F 0 "#PWR32" H 9475 1010 30  0001 C CNN
+F 0 "#PWR042" H 9475 1010 30  0001 C CNN
 F 1 "+3.3V" H 9475 1160 30  0000 C CNN
 	1    9475 1050
@@
 P 7875 1475
 F 0 "R4" V 7955 1475 50  0000 C CNN
-F 1 "50K" V 7875 1475 50  0000 C CNN
+F 1 "47K" V 7875 1475 50  0000 C CNN
 F 2 "R4" H 7875 1475 60  0001 C CNN
 	1    7875 1475
